File: star.kicad_sch (KiCad schematic)
At the start: 7 parts, among them J1 Conn_01x04_Pin, J2 Conn_01x08_Pin, SW1 SW_Push, SW2 SW_Push, U1 DHT11, U2 XIAO-ESP32-C3-SMD

Commit message: Swapped DHT11 for DS3231MZ
Parts:
- removed R1: 10000, Resistor_THT:R_Axial_DIN0204_L3.6mm_D1.6mm_P7.62mm_Horizontal, symbol Device:R
- removed U1: DHT11, Sensor:Aosong_DHT11_5.5x12.0_P2.54mm, symbol Sensor:DHT11
- added U1: DS3231MZ, Package_SO:SOIC-8_3.9x4.9mm_P1.27mm, symbol Timer_RTC:DS3231MZ
Connections:
- net +3.3V: now also J1.2 (Pin_2), U2.12 (3V3_OUT), U1.2 (VCC); no longer J1.3 (Pin_3)
- net GND: now also J1.1 (Pin_1), U1.5 (GND); no longer J1.4 (Pin_4)
- net SCL: now also J1.3 (Pin_3), U1.8 (SCL); no longer J1.2 (Pin_2)
- net SDA: now also J1.4 (Pin_4), U1.7 (SDA); no longer J1.1 (Pin_1)
- no-connect marks 17 -> 21
Other:
- moved on the sheet: J1
